Commit message: backup

File: src/ashwini/urdf/ashwini.xacro (robot description, xacro)
@@ -2,11 +2,11 @@
 <robot name="ashwini" xmlns:xacro="ashwini_description_xacro_namespace">
   <!-- Dummy root link without inertia -->
-  <link name="dummy_root">
-  </link>
-  <joint name="dummy_root_to_base" type="fixed">
+  <!-- <link name="dummy_root">
+  </link> -->
+  <!-- <joint name="dummy_root_to_base" type="fixed">
     <parent link="dummy_root"/>
     <child link="base_link"/>
     <origin xyz="0 0 0" rpy="0 0 0"/>
-  </joint>
+  </joint> -->
   <xacro:include filename="$(find ashwini)/urdf/ashwini.gazebo" />
   <xacro:property name="pi" value="3.1415926535897931" />

Commit message: added rplidar and realsense in simulation

File: src/ashwini/urdf/ashwini.xacro (robot description, xacro)
@@ -4,5 +4,4 @@
   <xacro:include filename="$(find ashwini)/urdf/ashwini.gazebo" />
   <xacro:property name="pi" value="3.1415926535897931" />
-  <xacro:property name="camera_mass" value="0.1"/>
 	<xacro:property name="hokoyu_mass" value="1e-5"/>
   <xacro:property name="base_link_length_width_height" value="0.650 0.381 0.132" />
@@ -212,27 +211,4 @@
     <origin xyz="-0.037 0 -0.10785"/>
   </xacro:continuous_joint>
-  <link name="camera">
-		<inertial>
-			<mass value="${camera_mass}"/>
-			<origin xyz="0 0 0" rpy="0 0 0"/>
-			<inertia
-		        ixx="1e-6" ixy="0.0" ixz="0.0"
-		        iyy="1e-6" iyz="0.0"
-		        izz="1e-6"
-		      />
-		</inertial>
-		<visual>
-			<origin xyz="0 0 0" rpy="0 0 0"/>
-			<geometry>
-				<box size="0.05 0.05 0.05"/>
-			</geometry>
-		</visual>
-		<collision>
-			<origin xyz="0 0 0" rpy="0 0 0"/>
-			<geometry>
-				<box size="0.05 0.05 0.05"/>
-			</geometry>
-		</collision>
-	</link>
   <link name="hokuyo">
 		<inertial>
@@ -258,10 +234,4 @@
 		</collision>
 	</link>
-  <joint name="camera_joint" type="fixed">
-		<origin xyz="0.006 -0.2 0.4" rpy="0 0.2 0" />
-		<parent link="base_link"/>
-		<child link="camera" />
-		<axis xyz="0 1 0"/>
-	</joint>
 	<!-- Hokoyu Joint -->
 	<joint name="hokuyo_joint" type="fixed">
@@ -300,3 +270,9 @@
     <origin xyz="-0.2 -0.2 0.144" rpy="0 0 0"/>
   </joint>
+  <!-- Add this to your robot's URDF -->
+  <xacro:include filename="$(find realsense2_description)/urdf/_d435.urdf.xacro"/>
+  <xacro:include filename="$(find realsense2_description)/urdf/_d435.gazebo.xacro"/>
+  <xacro:sensor_d435 name="camera" parent="base_link" topics_ns="camera">
+      <origin xyz="0.2 -0.23 0.3" rpy="0 0 0"/>  <!-- Adjust position as needed -->
+  </xacro:sensor_d435>
 </robot>

Commit message: real test

File: src/ashwini/urdf/ashwini.xacro (robot description, xacro)
@@ -2,6 +2,13 @@
 <robot name="ashwini" xmlns:xacro="ashwini_description_xacro_namespace">
   <!-- Dummy root link without inertia -->
-  <xacro:include filename="$(find ashwini)/urdf/ashwini.gazebo" />
-  <xacro:property name="pi" value="3.1415926535897931" />
+  <!-- base_footprint is a virtual frame at the ground contact point -->
+  <link name="base_footprint" />
+  <joint name="base_footprint_joint" type="fixed">
+    <parent link="base_footprint" />
+    <child link="base_link" />
+    <!-- Adjust Z as needed (e.g., half the wheel radius or chassis height) -->
+    <origin xyz="0 0 0.216" rpy="0 0 0" />
+  </joint>
+  <!-- <xacro:include filename="$(find ashwini)/urdf/ashwini.gazebo" /> -->
   <xacro:property name="camera_mass" value="0.1"/>
 	<xacro:property name="hokoyu_mass" value="1e-5"/>
@@ -213,26 +220,31 @@
   </xacro:continuous_joint>
   <link name="camera">
-		<inertial>
-			<mass value="${camera_mass}"/>
-			<origin xyz="0 0 0" rpy="0 0 0"/>
-			<inertia
-		        ixx="1e-6" ixy="0.0" ixz="0.0"
-		        iyy="1e-6" iyz="0.0"
-		        izz="1e-6"
-		      />
-		</inertial>
-		<visual>
-			<origin xyz="0 0 0" rpy="0 0 0"/>
-			<geometry>
-				<box size="0.05 0.05 0.05"/>
-			</geometry>
-		</visual>
-		<collision>
-			<origin xyz="0 0 0" rpy="0 0 0"/>
-			<geometry>
-				<box size="0.05 0.05 0.05"/>
-			</geometry>
-		</collision>
-	</link>
+    <inertial>
+      <mass value="${camera_mass}"/>
+      <origin xyz="0 0 0" rpy="0 0 0"/>
+      <inertia
+        ixx="1e-6" ixy="0.0" ixz="0.0"
+        iyy="1e-6" iyz="0.0"
+        izz="1e-6"/>
+    </inertial>
+    <visual>
+      <geometry>
+        <box size="0.05 0.05 0.05"/>
+      </geometry>
+      <origin xyz="0 0 0" rpy="0 0 0"/>
+    </visual>
+    <collision>
+      <geometry>
+        <box size="0.05 0.05 0.05"/>
+      </geometry>
+      <origin xyz="0 0 0" rpy="0 0 0"/>
+    </collision>
+  </link>
+  <joint name="camera_joint" type="fixed">
+		<origin xyz="0.006 -0.2 0.4" rpy="0 0.2 0" />
+		<parent link="base_link"/>
+		<child link="camera" />
+		<axis xyz="0 1 0"/>
+	</joint>
   <link name="hokuyo">
 		<inertial>
@@ -258,13 +270,7 @@
 		</collision>
 	</link>
-  <joint name="camera_joint" type="fixed">
-		<origin xyz="0.006 -0.2 0.4" rpy="0 0.2 0" />
-		<parent link="base_link"/>
-		<child link="camera" />
-		<axis xyz="0 1 0"/>
-	</joint>
 	<!-- Hokoyu Joint -->
 	<joint name="hokuyo_joint" type="fixed">
-	    <origin xyz="0.001 -0.2 0.2" rpy="0 0 0" />
+	    <origin xyz="0.001 -0.2 0.2" rpy="0 0 3.1415592653589793238" />
 	    <parent link="base_link"/>
 	    <child link="hokuyo" />
@@ -300,3 +306,9 @@
     <origin xyz="-0.2 -0.2 0.144" rpy="0 0 0"/>
   </joint>
+  <link name="odom"/>
+  <joint name="odom_to_base" type="fixed">
+    <parent link="odom"/>
+    <child link="base_footprint"/>
+    <origin xyz="0 0 0" rpy="0 0 0"/>
+  </joint>
 </robot>

Commit message: switched to realsense

File: src/ashwini/urdf/ashwini.xacro (robot description, xacro)
@@ -2,7 +2,6 @@
 <robot name="ashwini" xmlns:xacro="ashwini_description_xacro_namespace">
   <!-- Dummy root link without inertia -->
-  <xacro:include filename="$(find ashwini)/urdf/ashwini.gazebo" />
-  <xacro:property name="pi" value="3.1415926535897931" />
-  <xacro:property name="camera_mass" value="0.1"/>
+  <!-- <xacro:include filename="$(find ashwini)/urdf/ashwini.gazebo" /> -->
+  <!-- <xacro:property name="pi" value="3.1415926535897931" /> -->
 	<xacro:property name="hokoyu_mass" value="1e-5"/>
   <xacro:property name="base_link_length_width_height" value="0.650 0.381 0.132" />
@@ -181,5 +180,5 @@
   <!--right_caster_plate_link is a well named link :-) -->
   <xacro:box_link link_name="right_castor_mount" length="${castor_mount_link_length}"
-                                                 width="${castor_mount_link_width}"
+                                                 width ="${castor_mount_link_width}"
                                                  height="${castor_mount_link_height}"
                                                  mass="${castor_mount_link_mass}">
@@ -212,27 +211,4 @@
     <origin xyz="-0.037 0 -0.10785"/>
   </xacro:continuous_joint>
-  <link name="camera">
-		<inertial>
-			<mass value="${camera_mass}"/>
-			<origin xyz="0 0 0" rpy="0 0 0"/>
-			<inertia
-		        ixx="1e-6" ixy="0.0" ixz="0.0"
-		        iyy="1e-6" iyz="0.0"
-		        izz="1e-6"
-		      />
-		</inertial>
-		<visual>
-			<origin xyz="0 0 0" rpy="0 0 0"/>
-			<geometry>
-				<box size="0.05 0.05 0.05"/>
-			</geometry>
-		</visual>
-		<collision>
-			<origin xyz="0 0 0" rpy="0 0 0"/>
-			<geometry>
-				<box size="0.05 0.05 0.05"/>
-			</geometry>
-		</collision>
-	</link>
   <link name="hokuyo">
 		<inertial>
@@ -258,45 +234,24 @@
 		</collision>
 	</link>
-  <joint name="camera_joint" type="fixed">
-		<origin xyz="0.006 -0.2 0.4" rpy="0 0.2 0" />
-		<parent link="base_link"/>
-		<child link="camera" />
-		<axis xyz="0 1 0"/>
-	</joint>
 	<!-- Hokoyu Joint -->
 	<joint name="hokuyo_joint" type="fixed">
-	    <origin xyz="0.001 -0.2 0.2" rpy="0 0 0" />
+	    <origin xyz="0.001 -0.2 0.2" rpy="0 3.14 0" />
 	    <parent link="base_link"/>
 	    <child link="hokuyo" />
 	    <axis xyz="0 1 0"/>
 	</joint>
-    <!-- IMU Sensor -->
-  <link name="imu_link">
-    <inertial>
-      <mass value="0.05"/>
-      <origin xyz="0 0 0" rpy="0 0 0"/>
-      <inertia ixx="0.0001" ixy="0.0" ixz="0.0"
-               iyy="0.0001" iyz="0.0"
-               izz="0.0001"/>
-    </inertial>
-    <visual>
-      <geometry>
-        <box size="0.05 0.05 0.02"/>
-      </geometry>
-      <material name="Blue">
-        <color rgba="0.0 0.0 1.0 1.0"/>
-      </material>
-    </visual>
-    <collision>
-      <geometry>
-        <box size="0.05 0.05 0.02"/>
-      </geometry>
-    </collision>
-  </link>
-  <!-- IMU Joint (Attach to Base Link) -->
-  <joint name="imu_joint" type="fixed">
+  <!-- Add this to your robot's URDF -->
+  <xacro:include filename="$(find realsense2_description)/urdf/_d455.urdf.xacro"/>
+  <!-- <xacro:include filename="$(find realsense2_description)/urdf/_d455.gazebo.xacro"/> -->
+  <xacro:sensor_d455 name="camera" parent="base_link">
+      <origin xyz="0.2 0 0.3" rpy="0 0 0"/>  <!-- Adjust position as needed -->
+  </xacro:sensor_d455>
+  <!-- <link name="camera_imu_optical_frame"/>
+d
+  <joint name="camera_imu_optical_joint" type="fixed">
     <parent link="base_link"/>
-    <child link="imu_link"/>
-    <origin xyz="-0.2 -0.2 0.144" rpy="0 0 0"/>
-  </joint>
+    <child link="camera_imu_optical_frame"/>
+    <origin xyz="0.15 0 0.10" rpy="1.5708 0 1.5708"/>
+    <axis xyz="0 0 1" rpy="0 0 0"/>
+</joint> -->
 </robot>

Commit message: updated motor control

File: src/ashwini/urdf/ashwini.xacro (robot description, xacro)
@@ -236,5 +236,5 @@
 	<!-- Hokoyu Joint -->
 	<joint name="hokuyo_joint" type="fixed">
-	    <origin xyz="0.001 -0.2 0.2" rpy="0 3.14 0" />
+	    <origin xyz="0.001 -0.2 0.2" rpy="3.14 3.14 0" />
 	    <parent link="base_link"/>
 	    <child link="hokuyo" />
